File: eagle/tree2023.brd (EAGLE design)
At the start: 65.7 x 88.5 mm, 56 parts

Commit message: pcb files update
Parts:
- removed R10, R11, R12, R13, R14, R15, R16, R17, R18, R3, R4, R5, R6, R7, R8, R9: (no value), 0my:R0603
Connections:
- net GND: no longer R10.2, R11.2, R12.2, R13.2, R14.2, R15.2, R16.2, R17.2, R18.2, R3.2, R4.2, R5.2, R6.2, R7.2, R8.2, R9.2
- net LED5V: no longer R3.1
- net N$1: no longer R4.1
- net N$10: no longer R13.1
- net N$11: no longer R14.1
- net N$12: no longer R15.1
- net N$13: no longer R16.1
- net N$14: no longer R17.1
- net N$15: no longer R18.1
- net N$2: no longer R5.1
- net N$3: no longer R6.1
- net N$4: no longer R7.1
- net N$5: no longer R8.1
- net N$6: no longer R9.1
- net N$7: no longer R10.1
- net N$8: no longer R11.1
- net N$9: no longer R12.1
Routing:
- net GND: track 43.7 -> 14.1 mm
- net N$5: track 12.1 -> 7.78 mm
- net N$15: track 14.8 -> 12.6 mm
- net N$8: track 6.57 -> 4.54 mm
- net N$7: track 6.54 -> 4.51 mm
- net N$6: track 6.53 -> 4.50 mm
- net N$11: track 6.75 -> 4.72 mm
- net N$9: track 14.0 -> 12.0 mm
- net N$10: track 6.68 -> 4.65 mm
- net N$13: track 6.44 -> 4.53 mm
- net N$14: track 14.2 -> 13.3 mm
- net N$2: track 6.54 -> 5.66 mm
- net N$3: track 6.81 -> 5.94 mm
- net N$1: track 6.71 -> 5.87 mm
- net LED5V: track 40.4 -> 39.6 mm
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Other:
- board text added: "XmasTree 2023 v0.3@TripArts Music"
- board text removed: "XmasTree 2023 v0.2@TripArts Music"
